File: VFDClock.sch (KiCad schematic (older format))
At the start: 8 parts, among them P1 Power, P2 Analog, P3 Digital, P4 Digital, P5 CONN_01X01, P6 CONN_01X01, P7 CONN_01X01, P8 CONN_01X01

Commit message: VFDとICをつないだ回路を作成
Parts:
- removed P5, P6, P7, P8: CONN_01X01, Socket_Arduino_Uno:Arduino_1pin, symbol Connector_Generic:Conn_01x01
- added C1: 0.1u, Capacitor_THT:C_Disc_D10.0mm_W2.5mm_P5.00mm, symbol Device:C
- added J1: Barrel_Jack_MountingPin, #MyFootPrints:DCJack_MJ-179PH, symbol Connector:Barrel_Jack_MountingPin
- added Q1, Q2, Q3, Q4, Q5, Q6: VFD_LD8035E, #MyFootPrints:VFD_LD8035E, symbol MyParts:VFD_LD8035E
- added R1, R2: 4.7k, Resistor_THT:R_Axial_DIN0207_L6.3mm_D2.5mm_P7.62mm_Horizontal, symbol Device:R
- added R3, R4, R5, R6, R7, R8: 560, Resistor_THT:R_Axial_DIN0207_L6.3mm_D2.5mm_P7.62mm_Horizontal, symbol Device:R
- added U1: IC_HT16K33, #MyFootPrints:IC_HT16K33, symbol MyParts:IC_HT16K33
Connections:
- net labels added: +12V, A4, A5, a, b, c, d, dp, e, f, g
- net labels removed: +3.3V
- wire segments 38 -> 132
- no-connect marks 5 -> 42
Other:
- note removed: "Holes"
